File: board/board.kicad_pcb (KiCad board)
At the start: 2 copper layers, 21 x 13 mm, 1 part

Commit message: Initial design
Parts:
- added C1: 4.7pF, Capacitor_SMD:C_0402_1005Metric, F.Cu at (152.8, 95.1)
- added C2: TPSE107K016R0100, stpup:CAPMP7344X43-T_V, F.Cu at (148.5, 97.4)
- added C3: TPSE107K016R0100, stpup:CAPMP7344X43-T_V, F.Cu at (166.9, 91.3)
- added C4: 100nF, Capacitor_SMD:C_0402_1005Metric, F.Cu at (159.2, 93.6)
- added C5: 100nF, Capacitor_SMD:C_0402_1005Metric, F.Cu at (155.6, 99.1)
- added C6: 100nF, Capacitor_SMD:C_0402_1005Metric, F.Cu at (154.6, 99.1)
- added C7: 33pF, Capacitor_SMD:C_0603_1608Metric, F.Cu at (160.7, 98.8)
- added D1: PMEG100V100ELPDAZ, stpup:PMEG100V100ELPDAZ, F.Cu at (162.2, 92.2)
- added FB1: 200R_2A, Inductor_SMD:L_0805_2012Metric, F.Cu at (168.8, 100.6)
- added FB2: 200R_2A, Inductor_SMD:L_0805_2012Metric, F.Cu at (168.8, 98.0)
- added J1: 022_battery_cells, on_edge:debug_edge_2x05_device, F.Cu at (140.0, 96.5)
- added J2: 011_GPIO, on_edge:debug_edge_2x05_host, F.Cu at (176.3, 96.5)
- added L1: 4.7uH, stpup:WURTH 5040, F.Cu at (155.2, 88.7)
- added R1: 160 kOhms, Resistor_SMD:R_0603_1608Metric, F.Cu at (160.7, 100.3)
- added R2: 75 kOhms, Resistor_SMD:R_0603_1608Metric, F.Cu at (151.5, 97.6)
- added R4: 22 kOhms, Resistor_SMD:R_0603_1608Metric, F.Cu at (153.0, 97.6)
- added R5: 100 kOhms, Resistor_SMD:R_0603_1608Metric, F.Cu at (156.9, 99.6)
- added R6: 6.2 kOhms, Resistor_SMD:R_0603_1608Metric, F.Cu at (158.5, 99.5)
- added U1: LM2623LDX/NOPB, stpup:NHE0014A_V, F.Cu at (156.0, 95.2)
- moved LOGO1 12.1 mm to (144.2, 88.4)
Routing:
- net /stepup_2-LR6/VDD: track 0.00 -> 41.3 mm, vias 0 -> 2
- net /stepup_2-LR6/VIN: track 0.00 -> 22.4 mm, vias 0 -> 1
- net GND: track 0.00 -> 16.3 mm, vias 0 -> 160
- net /stepup_2-LR6/SW: track 0.00 -> 15.1 mm
- net /stepup_2-LR6/FREQ: track 0.00 -> 7.54 mm, vias 0 -> 2
- net /stepup_2-LR6/FB: track 0.00 -> 5.58 mm
- net /stepup_2-LR6/3.3V: track 0.00 -> 4.19 mm
- net /stepup_2-LR6/5V: track 0.00 -> 3.35 mm, vias 0 -> 1
- net Net-(R1-Pad1): track 0.00 -> 1.51 mm
- net Net-(C1-Pad1): track 0.00 -> 1.49 mm
- net /stepup_2-LR6/HEATSINK: vias 0 -> 5
- added copper zone on B.Cu, net /stepup_2-LR6/HEATSINK
- added copper zone on B.Cu, net GND
- added copper zone on F.Cu, net GND
- added copper zone on In1.Cu, net GND
- added copper zone on In2.Cu, net GND
Other:
- board size 21 x 13 mm -> 36.4 x 18 mm
- copper layers 2 -> 4
- board text added: "b132_step-up_2cell_v0.1"
- board text added: "osf.011_gpio"
- board text added: "osf.022_bat"
